File: aurora_hw/led_controller.kicad_pcb (KiCad board)
At the start: 2 copper layers, 88.9 x 46.2 mm, 83 parts, among them J1 Screw_Terminal_01x02, J10 Conn_01x03, J2 SJ-3524-SMT, J3 Conn_01x03, J4 Conn_01x03, J5 Conn_01x03, J6 Conn_01x03, J7 Conn_01x03, J8 Conn_01x03, J9 Conn_01x03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

Commit message: Add switch for changing A/R ratio, lengthen DFN pads
Parts:
- added SW2: CL-SB-13A-01T, SP3T-CL-SB-13A-01T:CL-SB-13A-01T, F.Cu at (175.6, 103.9)
- C12: value 1u -> 2.2u
- R3: value 2.21k -> 2.2k
- U2: value 74HCT245 -> 74HCT245PW
- moved MK1 4.70 mm to (167.5, 107.1), turned to 0 degrees
- moved R22 2.68 mm to (160.6, 110.1)
- moved C2 2.08 mm to (161.7, 111.5), turned to 0 degrees
- moved R3 1.86 mm to (166.1, 111.1)
- moved C5 1.81 mm to (166.6, 106.9), turned to 90 degrees
- moved R21 1.42 mm to (162.8, 110.1), turned to -90 degrees
- moved C3 1.14 mm to (165.9, 103.9)
- moved U1 0.92 mm to (160.5, 105.4)
- moved kibuzzard-62AD5F34 0.51 mm to (96.5, 105.9)
- moved C12 0.34 mm to (155.8, 105.0)
Connections:
- U1 pad 9: GND -> /MIC_A/R
Routing:
- net +3V3: track 127.5 -> 149.1 mm
- net /MIC_A/R: track 0.00 -> 13.4 mm, vias 0 -> 1
- net /MIC_BIAS: track 5.94 -> 8.94 mm
- net Net-(C3-Pad2): track 12.9 -> 9.92 mm
- net Net-(C4-Pad1): track 1.77 -> 3.65 mm
- net /MIC_GAIN: track 18.0 -> 19.8 mm
- net Net-(C5-Pad2): track 2.59 -> 4.33 mm
- net /AUD_L: track 7.92 -> 9.43 mm
- net /AGC_THRESH: track 4.82 -> 5.77 mm
- net Net-(C6-Pad2): track 4.64 -> 5.45 mm
- net /MIC_ADC: track 6.72 -> 7.23 mm
- net /AUD_L_ADC: track 14.6 -> 14.1 mm
- net GND: vias 175 -> 179
