File: aurora_hw/led_controller.kicad_pcb (KiCad board)
At the start: 2 copper layers, 88.9 x 46.2 mm, 84 parts, among them J1 Screw_Terminal_01x02, J10 Conn_01x03, J2 SJ-3524-SMT, J3 Conn_01x03, J4 Conn_01x03, J5 Conn_01x03, J6 Conn_01x03, J7 Conn_01x03, J8 Conn_01x03, J9 Conn_01x03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

Commit message: Hardware v2
Parts:
- C12: value 2.2u -> 1u
- C3: value 0.1u -> 10u
- moved C9 0.27 mm to (159.0, 98.3)
- moved C10 0.09 mm to (159.0, 92.5)
Connections:
- SW2 pad 1: unconnected-(SW2-Pad1) -> +3V3
- SW2 pad 2: +3V3 -> GND
- SW2 pad 3: /MIC_A/R -> /MIC_GAIN
- SW2 pad 4: GND -> unconnected-(SW2-Pad4)
- U3 pad 27: /MIC_GAIN -> /MIC_A/R
Routing:
- net /MIC_GAIN: track 19.8 -> 13.2 mm, vias 0 -> 1
- net /MIC_A/R: track 13.4 -> 19.7 mm, vias 1 -> 0
- net +3V3: track 149.1 -> 153.2 mm
- net GND: vias 179 -> 176
Other:
- board text added: "GAIN"
